Commit message: now rewards will be changed

File: resources/robots/bolt6/urdf/bolt6.urdf (robot description, URDF)
Before this commit: robot bolt, 9 links, 8 joints
Joints:
- joint FL_ANKLE: limit lower=-1 upper=1 effort=2.5 velocity=50 -> lower=-1 upper=1 effort=2.5 velocity=20
- joint FL_HAA: limit lower=-0.36 upper=1.0472 effort=2.5 velocity=50 -> lower=-0.36 upper=1.0472 effort=2.5 velocity=20
- joint FL_HFE: limit lower=-1.57 upper=1.57 effort=2.5 velocity=50 -> lower=-1.57 upper=1.57 effort=2.5 velocity=20
- joint FL_KFE: limit lower=-3.14 upper=0.0 effort=2.5 velocity=50 -> lower=-3.14 upper=0.0 effort=2.5 velocity=20
- joint FR_ANKLE: limit lower=-1 upper=1 effort=2.5 velocity=50 -> lower=-1 upper=1 effort=2.5 velocity=20
- joint FR_HAA: limit lower=-1.0472 upper=0.36 effort=2.5 velocity=50 -> lower=-1.0472 upper=0.36 effort=2.5 velocity=20
- joint FR_HFE: limit lower=-1.57 upper=1.57 effort=2.5 velocity=50 -> lower=-1.57 upper=1.57 effort=2.5 velocity=20
- joint FR_KFE: limit lower=-3.14 upper=0.0 effort=2.5 velocity=50 -> lower=-3.14 upper=0.0 effort=2.5 velocity=20

Commit message: bolt_walking

File: resources/robots/bolt6/urdf/bolt6.urdf (robot description, URDF)
Before this commit: robot bolt, 9 links, 8 joints
Joints:
- joint FL_ANKLE: limit lower=-1 upper=1 effort=2.5 velocity=20 -> lower=-1 upper=1 effort=2.5 velocity=15
- joint FL_HAA: limit lower=-0.36 upper=1.0472 effort=2.5 velocity=20 -> lower=-0.36 upper=1.0472 effort=2.5 velocity=15
- joint FL_HFE: limit lower=-1.57 upper=1.57 effort=2.5 velocity=20 -> lower=-1.57 upper=1.57 effort=2.5 velocity=15
- joint FL_KFE: limit lower=-3.14 upper=0.0 effort=2.5 velocity=20 -> lower=-3.14 upper=0.0 effort=2.5 velocity=15
- joint FR_ANKLE: limit lower=-1 upper=1 effort=2.5 velocity=20 -> lower=-1 upper=1 effort=2.5 velocity=15
- joint FR_HAA: limit lower=-1.0472 upper=0.36 effort=2.5 velocity=20 -> lower=-1.0472 upper=0.36 effort=2.5 velocity=15
- joint FR_HFE: limit lower=-1.57 upper=1.57 effort=2.5 velocity=20 -> lower=-1.57 upper=1.57 effort=2.5 velocity=15
- joint FR_KFE: limit lower=-3.14 upper=0.0 effort=2.5 velocity=20 -> lower=-3.14 upper=0.0 effort=2.5 velocity=15
